Commit message: Aktualizovanie .urdf súborov na základe aktuálneho .sdf

File: src/jetbot_description/models/urdf/jetbot.urdf (robot description, URDF)
Before this commit: robot jetbot, 8 links, 7 joints
Links:
- added link antenna_1, mass 0.02; collision cylinder length=0.15 radius=0.005; visual cylinder length=0.15 radius=0.005
- added link antenna_2, mass 0.02; collision cylinder length=0.15 radius=0.005; visual cylinder length=0.15 radius=0.005
- added link balance_wheel_2_base, mass 0.01; collision box size=0.02 0.02 0.02; visual box size=0.02 0.02 0.02
- added link balance_wheel_base, mass 0.01; collision box size=0.02 0.02 0.02; visual box size=0.02 0.02 0.02
- added link battery_1, mass 0.05; collision cylinder length=0.050 radius=0.009; visual cylinder length=0.050 radius=0.009
- added link battery_2, mass 0.05; collision cylinder length=0.050 radius=0.009; visual cylinder length=0.050 radius=0.009
- added link battery_3, mass 0.05; collision cylinder length=0.050 radius=0.009; visual cylinder length=0.050 radius=0.009
- added link camera_base, mass 0.05; collision box size=0.015 0.010 0.04; visual box size=0.015 0.010 0.04
- added link jetson_nano, mass 0.2; collision box size=0.08 0.08 0.014; visual box size=0.08 0.08 0.014
- added link motherboard, mass 0.2; collision box size=0.08 0.08 0.009; visual box size=0.08 0.08 0.009
- added link pillar_1, mass 0.05; collision cylinder length=0.05 radius=0.005; visual cylinder length=0.05 radius=0.005
- added link pillar_2, mass 0.05; collision cylinder length=0.05 radius=0.005; visual cylinder length=0.05 radius=0.005
- added link pillar_3, mass 0.05; collision cylinder length=0.05 radius=0.005; visual cylinder length=0.05 radius=0.005
- added link pillar_4, mass 0.05; collision cylinder length=0.05 radius=0.005; visual cylinder length=0.05 radius=0.005
- added link pillar_5, mass 0.02; collision cylinder length=0.025 radius=0.005; visual cylinder length=0.025 radius=0.005
- added link pillar_6, mass 0.02; collision cylinder length=0.025 radius=0.005; visual cylinder length=0.025 radius=0.005
- added link pillar_7, mass 0.02; collision cylinder length=0.025 radius=0.005; visual cylinder length=0.025 radius=0.005
- added link pillar_8, mass 0.02; collision cylinder length=0.025 radius=0.005; visual cylinder length=0.025 radius=0.005
- added link plate, mass 0.1; collision box size=0.12 0.12 0.001; visual box size=0.12 0.12 0.001
- added link speaker, mass 0.01; collision cylinder length=0.004 radius=0.01; visual cylinder length=0.004 radius=0.01
- added link top_plate, mass 0.1; collision box size=0.12 0.12 0.005; visual box size=0.12 0.12 0.005
- link balance_wheel: geometry collision cylinder length=0.005 radius=0.009; visual cylinder length=0.005 radius=0.009
- link balance_wheel_2: geometry collision cylinder length=0.005 radius=0.009; visual cylinder length=0.005 radius=0.009
- link base_link: mass 1.5 -> 1.6
- link camera: geometry visual box size=0.02 0.02 0.02
- link lidar_base: geometry collision cylinder length=0.030 radius=0.04; visual cylinder length=0.030 radius=0.04
Joints:
- removed joint balance_joint
- removed joint balance_joint_2
- added joint antenna_1_joint: type fixed, parent base_link, child antenna_1, origin xyz=-0.08 0.04 0.09 rpy=0 0 0
- added joint antenna_2_joint: type fixed, parent base_link, child antenna_2, origin xyz=-0.08 -0.04 0.09 rpy=0 0 0
- added joint balance_wheel_2_base_joint: type continuous, parent base_link, child balance_wheel_2_base, origin xyz=-0.07 0 -0.034 rpy=0 0 0, axis 0 0 1
- added joint balance_wheel_2_joint: type continuous, parent balance_wheel_2_base, child balance_wheel_2, origin xyz=0 0 -0.01 rpy=1.5707 0 0, axis 0 0 1
- added joint balance_wheel_base_joint: type continuous, parent base_link, child balance_wheel_base, origin xyz=0.07 0 -0.034 rpy=0 0 0, axis 0 0 1
- added joint balance_wheel_joint: type continuous, parent balance_wheel_base, child balance_wheel, origin xyz=0 0 -0.01 rpy=1.5707 0 0, axis 0 0 1
- added joint battery_1_joint: type fixed, parent plate, child battery_1, origin xyz=-0.018 0 -0.010 rpy=1.5707 1.5707 0
- added joint battery_2_joint: type fixed, parent plate, child battery_2, origin xyz=0 0 -0.010 rpy=1.5707 1.5707 0
- added joint battery_3_joint: type fixed, parent plate, child battery_3, origin xyz=0.018 0 -0.010 rpy=1.5707 1.5707 0
- added joint camera_base_joint: type fixed, parent base_link, child camera_base, origin xyz=0.09 0 0.045 rpy=0 0 0
- added joint jetson_nano_joint: type fixed, parent top_plate, child jetson_nano, origin xyz=0 0 -0.005 rpy=0 0 0
- added joint motherboard_joint: type fixed, parent plate, child motherboard, origin xyz=0 0 0.005 rpy=0 0 0
- added joint pillar_1_joint: type fixed, parent base_link, child pillar_1, origin xyz=0.05 0.05 0.025 rpy=0 0 0
- added joint pillar_2_joint: type fixed, parent base_link, child pillar_2, origin xyz=-0.05 0.05 0.025 rpy=0 0 0
- added joint pillar_3_joint: type fixed, parent base_link, child pillar_3, origin xyz=0.05 -0.05 0.025 rpy=0 0 0
- added joint pillar_4_joint: type fixed, parent base_link, child pillar_4, origin xyz=-0.05 -0.05 0.025 rpy=0 0 0
- added joint pillar_5_joint: type fixed, parent plate, child pillar_5, origin xyz=0.045 0.045 0.0125 rpy=0 0 0
- added joint pillar_6_joint: type fixed, parent plate, child pillar_6, origin xyz=-0.045 0.045 0.0125 rpy=0 0 0
- added joint pillar_7_joint: type fixed, parent plate, child pillar_7, origin xyz=0.045 -0.045 0.0125 rpy=0 0 0
- added joint pillar_8_joint: type fixed, parent plate, child pillar_8, origin xyz=-0.045 -0.045 0.0125 rpy=0 0 0
- added joint plate_joint: type fixed, parent pillar_1, child plate, origin xyz=-0.05 -0.05 0.025 rpy=0 0 0
- added joint speaker_joint: type fixed, parent base_link, child speaker, origin xyz=-0.05 0.075 0.026 rpy=0 0 0
- added joint top_plate_joint: type fixed, parent pillar_5, child top_plate, origin xyz=-0.045 -0.045 0.0125 rpy=0 0 0
- joint camera_joint: origin xyz=0.1 0 0.03 rpy=0 0 0 -> xyz=0.01 0 0.025 rpy=0 0.15 0; parent base_link -> camera_base
- joint lidar_base_joint: origin xyz=0 0 0.025 rpy=0 0 0 -> xyz=0 0 0.010 rpy=0 0 0; parent base_link -> top_plate
- joint lidar_joint: origin xyz=0 0 0.035 rpy=0 0 0 -> xyz=0 0 0.025 rpy=0 0 0

File: src/jetbot_gazebo/models/jetbot/urdf/jetbot.urdf (robot description, URDF)
Before this commit: robot jetbot, 8 links, 7 joints
Links:
- added link antenna_1, mass 0.02; collision cylinder length=0.15 radius=0.005; visual cylinder length=0.15 radius=0.005
- added link antenna_2, mass 0.02; collision cylinder length=0.15 radius=0.005; visual cylinder length=0.15 radius=0.005
- added link balance_wheel_2_base, mass 0.01; collision box size=0.02 0.02 0.02; visual box size=0.02 0.02 0.02
- added link balance_wheel_base, mass 0.01; collision box size=0.02 0.02 0.02; visual box size=0.02 0.02 0.02
- added link battery_1, mass 0.05; collision cylinder length=0.050 radius=0.009; visual cylinder length=0.050 radius=0.009
- added link battery_2, mass 0.05; collision cylinder length=0.050 radius=0.009; visual cylinder length=0.050 radius=0.009
- added link battery_3, mass 0.05; collision cylinder length=0.050 radius=0.009; visual cylinder length=0.050 radius=0.009
- added link camera_base, mass 0.05; collision box size=0.015 0.010 0.04; visual box size=0.015 0.010 0.04
- added link jetson_nano, mass 0.2; collision box size=0.08 0.08 0.014; visual box size=0.08 0.08 0.014
- added link motherboard, mass 0.2; collision box size=0.08 0.08 0.009; visual box size=0.08 0.08 0.009
- added link pillar_1, mass 0.05; collision cylinder length=0.05 radius=0.005; visual cylinder length=0.05 radius=0.005
- added link pillar_2, mass 0.05; collision cylinder length=0.05 radius=0.005; visual cylinder length=0.05 radius=0.005
- added link pillar_3, mass 0.05; collision cylinder length=0.05 radius=0.005; visual cylinder length=0.05 radius=0.005
- added link pillar_4, mass 0.05; collision cylinder length=0.05 radius=0.005; visual cylinder length=0.05 radius=0.005
- added link pillar_5, mass 0.02; collision cylinder length=0.025 radius=0.005; visual cylinder length=0.025 radius=0.005
- added link pillar_6, mass 0.02; collision cylinder length=0.025 radius=0.005; visual cylinder length=0.025 radius=0.005
- added link pillar_7, mass 0.02; collision cylinder length=0.025 radius=0.005; visual cylinder length=0.025 radius=0.005
- added link pillar_8, mass 0.02; collision cylinder length=0.025 radius=0.005; visual cylinder length=0.025 radius=0.005
- added link plate, mass 0.1; collision box size=0.12 0.12 0.001; visual box size=0.12 0.12 0.001
- added link speaker, mass 0.01; collision cylinder length=0.004 radius=0.01; visual cylinder length=0.004 radius=0.01
- added link top_plate, mass 0.1; collision box size=0.12 0.12 0.005; visual box size=0.12 0.12 0.005
- link balance_wheel: geometry collision cylinder length=0.005 radius=0.009; visual cylinder length=0.005 radius=0.009
- link balance_wheel_2: geometry collision cylinder length=0.005 radius=0.009; visual cylinder length=0.005 radius=0.009
- link base_link: mass 1.5 -> 1.6
- link camera: geometry visual box size=0.02 0.02 0.02
- link lidar_base: geometry collision cylinder length=0.030 radius=0.04; visual cylinder length=0.030 radius=0.04
Joints:
- removed joint balance_joint
- removed joint balance_joint_2
- added joint antenna_1_joint: type fixed, parent base_link, child antenna_1, origin xyz=-0.08 0.04 0.09 rpy=0 0 0
- added joint antenna_2_joint: type fixed, parent base_link, child antenna_2, origin xyz=-0.08 -0.04 0.09 rpy=0 0 0
- added joint balance_wheel_2_base_joint: type continuous, parent base_link, child balance_wheel_2_base, origin xyz=-0.07 0 -0.034 rpy=0 0 0, axis 0 0 1
- added joint balance_wheel_2_joint: type continuous, parent balance_wheel_2_base, child balance_wheel_2, origin xyz=0 0 -0.01 rpy=1.5707 0 0, axis 0 0 1
- added joint balance_wheel_base_joint: type continuous, parent base_link, child balance_wheel_base, origin xyz=0.07 0 -0.034 rpy=0 0 0, axis 0 0 1
- added joint balance_wheel_joint: type continuous, parent balance_wheel_base, child balance_wheel, origin xyz=0 0 -0.01 rpy=1.5707 0 0, axis 0 0 1
- added joint battery_1_joint: type fixed, parent plate, child battery_1, origin xyz=-0.018 0 -0.010 rpy=1.5707 1.5707 0
- added joint battery_2_joint: type fixed, parent plate, child battery_2, origin xyz=0 0 -0.010 rpy=1.5707 1.5707 0
- added joint battery_3_joint: type fixed, parent plate, child battery_3, origin xyz=0.018 0 -0.010 rpy=1.5707 1.5707 0
- added joint camera_base_joint: type fixed, parent base_link, child camera_base, origin xyz=0.09 0 0.045 rpy=0 0 0
- added joint jetson_nano_joint: type fixed, parent top_plate, child jetson_nano, origin xyz=0 0 -0.005 rpy=0 0 0
- added joint motherboard_joint: type fixed, parent plate, child motherboard, origin xyz=0 0 0.005 rpy=0 0 0
- added joint pillar_1_joint: type fixed, parent base_link, child pillar_1, origin xyz=0.05 0.05 0.025 rpy=0 0 0
- added joint pillar_2_joint: type fixed, parent base_link, child pillar_2, origin xyz=-0.05 0.05 0.025 rpy=0 0 0
- added joint pillar_3_joint: type fixed, parent base_link, child pillar_3, origin xyz=0.05 -0.05 0.025 rpy=0 0 0
- added joint pillar_4_joint: type fixed, parent base_link, child pillar_4, origin xyz=-0.05 -0.05 0.025 rpy=0 0 0
- added joint pillar_5_joint: type fixed, parent plate, child pillar_5, origin xyz=0.045 0.045 0.0125 rpy=0 0 0
- added joint pillar_6_joint: type fixed, parent plate, child pillar_6, origin xyz=-0.045 0.045 0.0125 rpy=0 0 0
- added joint pillar_7_joint: type fixed, parent plate, child pillar_7, origin xyz=0.045 -0.045 0.0125 rpy=0 0 0
- added joint pillar_8_joint: type fixed, parent plate, child pillar_8, origin xyz=-0.045 -0.045 0.0125 rpy=0 0 0
- added joint plate_joint: type fixed, parent pillar_1, child plate, origin xyz=-0.05 -0.05 0.025 rpy=0 0 0
- added joint speaker_joint: type fixed, parent base_link, child speaker, origin xyz=-0.05 0.075 0.026 rpy=0 0 0
- added joint top_plate_joint: type fixed, parent pillar_5, child top_plate, origin xyz=-0.045 -0.045 0.0125 rpy=0 0 0
- joint camera_joint: origin xyz=0.1 0 0.03 rpy=0 0 0 -> xyz=0.01 0 0.025 rpy=0 0.15 0; parent base_link -> camera_base
- joint lidar_base_joint: origin xyz=0 0 0.025 rpy=0 0 0 -> xyz=0 0 0.010 rpy=0 0 0; parent base_link -> top_plate
- joint lidar_joint: origin xyz=0 0 0.035 rpy=0 0 0 -> xyz=0 0 0.025 rpy=0 0 0

Commit message: Vykonanie potrebných zmien pre aktualizovanie .urdf podľa aktuálne .sdf
- pridanie všetkých potrebných závislostí
- aktualizovanie aby bol kód rovnaký v .urdf
- aktualizovanie verzie

- ver: 0.63

File: src/jetbot_description/models/urdf/jetbot.urdf (robot description, URDF)
Before this commit: robot jetbot, 29 links, 28 joints
Links:
- link balance_wheel: geometry collision sphere radius=0.009; visual sphere radius=0.009
- link balance_wheel_2: geometry collision sphere radius=0.009; visual sphere radius=0.009
- link camera: mass None -> 0.05; geometry collision box size=0.02 0.02 0.02; visual box size=0.02 0.02 0.02
- link lidar: mass None -> 0.1; geometry collision cylinder length=0.02 radius=0.04; visual cylinder length=0.02 radius=0.04
Joints:
- joint balance_wheel_2_joint: axis 0 0 1 -> (none); type continuous -> fixed
- joint balance_wheel_joint: axis 0 0 1 -> (none); type continuous -> fixed
- joint plate_joint: origin xyz=-0.05 -0.05 0.025 rpy=0 0 0 -> xyz=0 0 0.050 rpy=0 0 0; parent pillar_1 -> base_link
- joint top_plate_joint: origin xyz=-0.045 -0.045 0.0125 rpy=0 0 0 -> xyz=0 0 0.025 rpy=0 0 0; parent pillar_5 -> plate

File: src/jetbot_gazebo/models/jetbot/urdf/jetbot.urdf (robot description, URDF)
Before this commit: robot jetbot, 29 links, 28 joints
Links:
- link balance_wheel: geometry collision sphere radius=0.009; visual sphere radius=0.009
- link balance_wheel_2: geometry collision sphere radius=0.009; visual sphere radius=0.009
- link camera: mass None -> 0.05; geometry collision box size=0.02 0.02 0.02; visual box size=0.02 0.02 0.02
- link lidar: mass None -> 0.1; geometry collision cylinder length=0.02 radius=0.04; visual cylinder length=0.02 radius=0.04
Joints:
- joint balance_wheel_2_joint: axis 0 0 1 -> (none); type continuous -> fixed
- joint balance_wheel_joint: axis 0 0 1 -> (none); type continuous -> fixed
- joint plate_joint: origin xyz=-0.05 -0.05 0.025 rpy=0 0 0 -> xyz=0 0 0.050 rpy=0 0 0; parent pillar_1 -> base_link
- joint top_plate_joint: origin xyz=-0.045 -0.045 0.0125 rpy=0 0 0 -> xyz=0 0 0.025 rpy=0 0 0; parent pillar_5 -> plate
